File: EasyDriver_v45/EasyDriver_v45.sch (EAGLE design)
At the start: 43 parts, among them IC1 A3967SLB, IC2 V_REG_317SMD

Commit message: Completed testing on first v4.5 prototypes, and wrote up results in notes.txt. Also added some text to schematic including formula for calculating Max Current from Vref voltage.
Other:
- note added: "At Vref of 1V max current will be 166mA"
- note added: "At Vref of 2V max current will be 333mA"
- note added: "At Vref of 5V max current will be 833mA"
- note added: "Max Coil Current(in Amps) = Vref(in Volts)/6"
- note added: "TP1 = Vref input to driver"
- note removed: "At VREF of 1V max current will be 166mA"
- note removed: "At VREF of 3.3V max current will be 550mA"
- note removed: "At VREF of 5V max current will be 833mA"
- note removed: "TP1 - VREF input to driver"
