File: Hardware/EasyDriver_v45.brd (EAGLE design)
At the start: 48.3 x 20.3 mm, 45 parts, among them IC1 A3967SLB, IC2 V_REG_317SMD

Commit message: Updating 2.4k to 2.49K resistor and updating to CC-SA 3.0
Parts:
- FRAME2: device SparkFun-Aesthetics:CREATIVE_COMMONS -> SparkFun-Retired:CREATIVE_COMMONS
- R5: value 2.4K -> 2.49K
- moved FRAME2 22.9 mm to (-5.08, -8.89)
Other:
- board text added: "Brian Schmalz"
- board text added: "Produced by SparkFun"
Changed lines of the file:
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@@
 <layer number="20" name="Dimension" color="15" fill="1" visible="yes" active="yes"/>
 <layer number="21" name="tPlace" color="16" fill="1" visible="yes" active="yes"/>
-<layer number="22" name="bPlace" color="14" fill="1" visible="no" active="yes"/>
+<layer number="22" name="bPlace" color="14" fill="1" visible="yes" active="yes"/>
 <layer number="23" name="tOrigins" color="15" fill="1" visible="yes" active="yes"/>
-<layer number="24" name="bOrigins" color="15" fill="1" visible="no" active="yes"/>
+<layer number="24" name="bOrigins" color="15" fill="1" visible="yes" active="yes"/>
 <layer number="25" name="tNames" color="7" fill="1" visible="no" active="yes"/>
 <layer number="26" name="bNames" color="7" fill="1" visible="no" active="yes"/>
@@
 <layer number="37" name="tTest" color="7" fill="1" visible="no" active="yes"/>
 <layer number="38" name="bTest" color="7" fill="1" visible="no" active="yes"/>
-<layer number="39" name="tKeepout" color="4" fill="11" visible="yes" active="yes"/>
+<layer number="39" name="tKeepout" color="4" fill="11" visible="no" active="yes"/>
 <layer number="40" name="bKeepout" color="1" fill="11" visible="no" active="yes"/>
 <layer number="41" name="tRestrict" color="4" fill="10" visible="no" active="yes"/>
@@
 <layer number="43" name="vRestrict" color="2" fill="10" visible="no" active="yes"/>
 <layer number="44" name="Drills" color="7" fill="1" visible="no" active="yes"/>
-<layer number="45" name="Holes" color="7" fill="1" visible="no" active="yes"/>
+<layer number="45" name="Holes" color="7" fill="1" visible="yes" active="yes"/>
 <layer number="46" name="Milling" color="3" fill="1" visible="no" active="yes"/>
 <layer number="47" name="Measures" color="7" fill="1" visible="no" active="yes"/>
 <layer number="48" name="Document" color="7" fill="1" visible="no" active="yes"/>
 <layer number="49" name="Reference" color="7" fill="1" visible="no" active="yes"/>
-<layer number="51" name="tDocu" color="6" fill="1" visible="no" active="yes"/>
+<layer number="51" name="tDocu" color="6" fill="1" visible="yes" active="yes"/>
 <layer number="52" name="bDocu" color="7" fill="1" visible="no" active="yes"/>
 <layer number="53" name="tGND_GNDA" color="7" fill="9" visible="no" active="yes"/>
@@
 <wire x1="8.382" y1="12.7" x2="9.398" y2="12.7" width="0.254" layer="21"/>
 <wire x1="9.398" y1="12.7" x2="9.017" y2="12.319" width="0.254" layer="21"/>
+<text x="25.4" y="-8.89" size="1.778" layer="51" font="vector" ratio="15">Brian Schmalz</text>
+<text x="6.35" y="-11.43" size="1.778" layer="51" font="vector" ratio="15">Produced by SparkFun</text>
 </plain>
 <attributes>
@@
 <attribute name="VALUE" x="45.063" y="9.84" size="0.6096" layer="27"/>
 </element>
-<element name="R5" library="SparkFun-Resistors" package="0603-RES" value="2.4K" x="5.08" y="17.78" smashed="yes" rot="R270">
+<element name="R5" library="SparkFun-Resistors" package="0603-RES" value="2.49K" x="5.08" y="17.78" smashed="yes" rot="R270">
 <attribute name="NAME" x="4.953" y="20.574" size="0.6096" layer="25"/>
 <attribute name="VALUE" x="4.953" y="19.558" size="0.6096" layer="27"/>
@@
 </element>
 <element name="TP1" library="SparkFun-Passives" package="TP_15TH" value="TEST-POINTTP_15TH_THRU" x="10.922" y="12.7"/>
-<element name="FRAME2" library="SparkFun-Aesthetics" package="CREATIVE_COMMONS" value="FRAME-LETTER" x="17.78" y="-10.16"/>
+<element name="FRAME2" library="SparkFun-Retired" package="CREATIVE_COMMONS" value="FRAME-LETTER" x="-5.08" y="-8.89"/>
 </elements>
 <signals>

Commit message: added regular fiducials
Parts:
- added FID1, FID2: FIDUCIAL1X2, SparkFun-Aesthetics:FIDUCIAL-1X2
